File: apple-1/chips/MMI-6301/kicad/prom_fpga.sch (KiCad schematic (older format))
At the start: 10 parts, among them U10 ICE40LP1K-CM36, U11 AT25DF041B

Commit message: MMI-6301 preliminary layout
Parts:
- removed TP4: TestPoint_Alt, prom:test-point-25, symbol Connector:TestPoint_Alt
- TP3, TP5, TP6, TP7, TP8: symbol Connector:TestPoint_Alt -> prom-rescue:TestPoint_Alt-Connector
Connections:
- net A0: now also U10.E2 (IOB_34); no longer U10.E1 (IOL_7B)
- net A3: now also U10.E1 (IOL_7B); no longer U10.E2 (IOB_34)
- no-connect marks 8 -> 9
Changed lines of the file:
@@
 A2
 Text GLabel 5300 4050 2    50   Input ~ 0
+A0
+Text GLabel 5300 5700 2    50   Input ~ 0
 A3
-Text GLabel 5300 5700 2    50   Input ~ 0
-A0
 Text GLabel 5300 5400 2    50   Input ~ 0
 A5
@@
 NoConn ~ 8800 5250
 $Comp
-L Connector:TestPoint_Alt TP4
-U 1 1 5E85122D
-P 7400 4100
-F 0 "TP4" H 7300 4350 50  0000 L CNN
-F 1 "TestPoint_Alt" H 7458 4127 50  0001 L CNN
-F 2 "prom:test-point-25" H 7600 4100 50  0001 C CNN
-F 3 "~" H 7600 4100 50  0001 C CNN
-	1    7400 4100
-	1    0    0    -1
-$EndComp
-$Comp
 L Device:R_US R2
 U 1 1 5E85311F
@@
 $EndComp
 $Comp
-L Connector:TestPoint_Alt TP6
+L prom-rescue:TestPoint_Alt-Connector TP6
 U 1 1 5E868480
 P 7500 4100
-F 0 "TP6" H 7500 4350 50  0000 L CNN
+AR Path="/5E868480" Ref="TP6"  Part="1"
+AR Path="/5E85CF8D/5E868480" Ref="TP5"  Part="1"
+F 0 "TP5" H 7500 4350 50  0000 L CNN
 F 1 "TestPoint_Alt" H 7558 4127 50  0001 L CNN
 F 2 "prom:test-point-25" H 7700 4100 50  0001 C CNN
@@
 $EndComp
 $Comp
-L Connector:TestPoint_Alt TP3
+L prom-rescue:TestPoint_Alt-Connector TP3
 U 1 1 5E86CD9D
 P 7300 5300
+AR Path="/5E86CD9D" Ref="TP3"  Part="1"
+AR Path="/5E85CF8D/5E86CD9D" Ref="TP3"  Part="1"
 F 0 "TP3" H 7350 5550 50  0000 R CNN
 F 1 "TestPoint_Alt" H 7358 5327 50  0001 L CNN
@@
 $EndComp
 $Comp
-L Connector:TestPoint_Alt TP5
+L prom-rescue:TestPoint_Alt-Connector TP5
 U 1 1 5E86D314
 P 7400 5300
-F 0 "TP5" H 7450 5650 50  0000 R CNN
+AR Path="/5E86D314" Ref="TP5"  Part="1"
+AR Path="/5E85CF8D/5E86D314" Ref="TP4"  Part="1"
+F 0 "TP4" H 7450 5650 50  0000 R CNN
 F 1 "TestPoint_Alt" H 7458 5327 50  0001 L CNN
 F 2 "prom:test-point-25" H 7600 5300 50  0001 C CNN
@@
 $EndComp
 $Comp
-L Connector:TestPoint_Alt TP7
+L prom-rescue:TestPoint_Alt-Connector TP7
 U 1 1 5E86D600
 P 7500 5300
-F 0 "TP7" H 7550 5550 50  0000 R CNN
+AR Path="/5E86D600" Ref="TP7"  Part="1"
+AR Path="/5E85CF8D/5E86D600" Ref="TP6"  Part="1"
+F 0 "TP6" H 7550 5550 50  0000 R CNN
 F 1 "TestPoint_Alt" H 7558 5327 50  0001 L CNN
 F 2 "prom:test-point-25" H 7700 5300 50  0001 C CNN
@@
 $EndComp
 $Comp
-L Connector:TestPoint_Alt TP8
+L prom-rescue:TestPoint_Alt-Connector TP8
 U 1 1 5E86D938
 P 7600 5300
-F 0 "TP8" H 7650 5650 50  0000 R CNN
+AR Path="/5E86D938" Ref="TP8"  Part="1"
+AR Path="/5E85CF8D/5E86D938" Ref="TP7"  Part="1"
+F 0 "TP7" H 7650 5650 50  0000 R CNN
 F 1 "TestPoint_Alt" H 7658 5327 50  0001 L CNN
 F 2 "prom:test-point-25" H 7800 5300 50  0001 C CNN
@@
 	7950 4050 7950 4500
 Wire Wire Line
-	7150 4400 7400 4400
-Wire Wire Line
-	7400 4400 7400 4100
-Wire Wire Line
 	7500 4100 7500 4500
 Connection ~ 7500 4500
@@
 NoConn ~ 5000 4250
 NoConn ~ 4950 5600
+NoConn ~ 7150 4400
 $EndSCHEMATC

Commit message: fold the rescued schematic symbols into the local library
Parts:
- TP3, TP5, TP6, TP7, TP8: symbol prom-rescue:TestPoint_Alt-Connector -> local:TestPoint_Alt
Changed lines of the file:
@@
 FPGA and SPI flash
 $Comp
-L power:GND #PWR026
+L local:GND #PWR026
 U 1 1 5E915F0B
 P 2650 5450
@@
 $EndComp
 $Comp
-L power:GND #PWR031
+L local:GND #PWR031
 U 1 1 5E91627E
 P 9450 5450
@@
 $EndComp
 $Comp
-L power:+3.3V #PWR025
+L local:+3.3V #PWR025
 U 1 1 5E91732E
 P 2650 4050
@@
 $EndComp
 $Comp
-L power:+1V2 #PWR027
+L local:+1V2 #PWR027
 U 1 1 5E917DDE
 P 2800 4950
@@
 $EndComp
 $Comp
-L power:+3.3V #PWR030
+L local:+3.3V #PWR030
 U 1 1 5E84E3FB
 P 9450 4550
@@
 	10400 4950 9950 4950
 $Comp
-L power:+3.3V #PWR029
+L local:+3.3V #PWR029
 U 1 1 5E85F98D
 P 8300 3750
@@
 $EndComp
 $Comp
-L power:+3.3V #PWR028
+L local:+3.3V #PWR028
 U 1 1 5E863EF8
 P 7950 3750
@@
 $EndComp
 $Comp
-L prom-rescue:TestPoint_Alt-Connector TP6
+L local:TestPoint_Alt TP6
 U 1 1 5E868480
 P 7500 4100
@@
 $EndComp
 $Comp
-L prom-rescue:TestPoint_Alt-Connector TP3
+L local:TestPoint_Alt TP3
 U 1 1 5E86CD9D
 P 7300 5300
@@
 $EndComp
 $Comp
-L prom-rescue:TestPoint_Alt-Connector TP5
+L local:TestPoint_Alt TP5
 U 1 1 5E86D314
 P 7400 5300
@@
 $EndComp
 $Comp
-L prom-rescue:TestPoint_Alt-Connector TP7
+L local:TestPoint_Alt TP7
 U 1 1 5E86D600
 P 7500 5300
@@
 $EndComp
 $Comp
-L prom-rescue:TestPoint_Alt-Connector TP8
+L local:TestPoint_Alt TP8
 U 1 1 5E86D938
 P 7600 5300
