File: apple-1/chips/MMI-6301/kicad/prom_fpga.sch (KiCad schematic (older format))
At the start: 9 parts, among them U10 ICE40LP1K-CM36, U11 AT25DF041B

Commit message: completed layout
Parts:
- TP3, TP5, TP6, TP7, TP8: footprint prom:test-point-25 -> prom:test-point
Changed lines of the file:
@@
 F 0 "TP5" H 6850 4250 50  0000 L CNN
 F 1 "TestPoint_Alt" H 6908 4027 50  0001 L CNN
-F 2 "prom:test-point-25" H 7050 4000 50  0001 C CNN
+F 2 "prom:test-point" H 7050 4000 50  0001 C CNN
 F 3 "~" H 7050 4000 50  0001 C CNN
 	1    6850 4000
@@
 F 0 "TP3" H 6700 5450 50  0000 R CNN
 F 1 "TestPoint_Alt" H 6708 5227 50  0001 L CNN
-F 2 "prom:test-point-25" H 6850 5200 50  0001 C CNN
+F 2 "prom:test-point" H 6850 5200 50  0001 C CNN
 F 3 "~" H 6850 5200 50  0001 C CNN
 	1    6650 5200
@@
 F 0 "TP4" H 6800 5550 50  0000 R CNN
 F 1 "TestPoint_Alt" H 6808 5227 50  0001 L CNN
-F 2 "prom:test-point-25" H 6950 5200 50  0001 C CNN
+F 2 "prom:test-point" H 6950 5200 50  0001 C CNN
 F 3 "~" H 6950 5200 50  0001 C CNN
 	1    6750 5200
@@
 F 0 "TP6" H 6900 5450 50  0000 R CNN
 F 1 "TestPoint_Alt" H 6908 5227 50  0001 L CNN
-F 2 "prom:test-point-25" H 7050 5200 50  0001 C CNN
+F 2 "prom:test-point" H 7050 5200 50  0001 C CNN
 F 3 "~" H 7050 5200 50  0001 C CNN
 	1    6850 5200
@@
 F 0 "TP7" H 7000 5550 50  0000 R CNN
 F 1 "TestPoint_Alt" H 7008 5227 50  0001 L CNN
-F 2 "prom:test-point-25" H 7150 5200 50  0001 C CNN
+F 2 "prom:test-point" H 7150 5200 50  0001 C CNN
 F 3 "~" H 7150 5200 50  0001 C CNN
 	1    6950 5200

Commit message: library tweak
Parts:
- R1, R2: symbol Device:R_US -> local:R_US
Changed lines of the file:
@@
 NoConn ~ 8150 5150
 $Comp
-L Device:R_US R2
+L local:R_US R2
 U 1 1 5E85311F
 P 7650 3800
@@
 $EndComp
 $Comp
-L Device:R_US R1
+L local:R_US R1
 U 1 1 5E855891
 P 7300 3800
