File: apple-1/chips/MMI-6301/kicad/prom_io_power.sch (KiCad schematic (older format))
At the start: 15 parts, among them J1 DIP16_pins, U1 TLV743P 3.3V, U2 TLV743P 1.2V, U3 74LVC2G34, U4 74LVC2G34, U5 74LVC2G34, U6 74LVC2G34, U7 74LVC2G34, U8 74LVC2G125, U9 74LVC2G125

Commit message: MMI-6301 preliminary layout
Parts:
- TP1, TP2: symbol Connector:TestPoint_Alt -> prom-rescue:TestPoint_Alt-Connector
Connections:
- wire segments 82 -> 86
Other:
- moved on the sheet: C3, TP2, U2
Changed lines of the file:
@@
 L local:TLV743P U2
 U 1 1 5E8089C0
-P 2200 6500
-F 0 "U2" H 2325 7315 50  0000 C CNN
-F 1 "TLV743P 1.2V" H 2325 7224 50  0000 C CNN
-F 2 "prom:X2SON" H 2200 6500 100 0001 C CNN
-F 3 "" H 2200 6500 100 0001 C CNN
-	1    2200 6500
+P 2200 6700
+F 0 "U2" H 2325 7515 50  0000 C CNN
+F 1 "TLV743P 1.2V" H 2325 7424 50  0000 C CNN
+F 2 "prom:X2SON" H 2200 6700 100 0001 C CNN
+F 3 "" H 2200 6700 100 0001 C CNN
+	1    2200 6700
 	1    0    0    -1
 $EndComp
@@
 DIP_A6
 Text Label 5000 5650 2    50   ~ 0
+DIP_CE1_N
+Text Label 5000 5750 2    50   ~ 0
 DIP_CE2_N
-Text Label 5000 5750 2    50   ~ 0
-DIP_CE1_N
 $Comp
 L local:74LVC2G34 U?
@@
 A6
 Text GLabel 6100 5650 2    50   Output ~ 0
+CE1_N
+Text GLabel 6100 5750 2    50   Output ~ 0
 CE2_N
-Text GLabel 6100 5750 2    50   Output ~ 0
-CE1_N
 Wire Notes Line
 	4550 6400 4550 6500
@@
 L power:+1V2 #PWR010
 U 1 1 5E84CCB2
-P 3450 5950
-F 0 "#PWR010" H 3450 5800 50  0001 C CNN
-F 1 "+1V2" H 3465 6123 50  0000 C CNN
-F 2 "" H 3450 5950 50  0001 C CNN
-F 3 "" H 3450 5950 50  0001 C CNN
-	1    3450 5950
+P 3450 6150
+F 0 "#PWR010" H 3450 6000 50  0001 C CNN
+F 1 "+1V2" H 3465 6323 50  0000 C CNN
+F 2 "" H 3450 6150 50  0001 C CNN
+F 3 "" H 3450 6150 50  0001 C CNN
+	1    3450 6150
 	1    0    0    -1
 $EndComp
@@
 L power:+3.3V #PWR09
 U 1 1 5E84D3A3
-P 3400 4900
-F 0 "#PWR09" H 3400 4750 50  0001 C CNN
-F 1 "+3.3V" H 3415 5073 50  0000 C CNN
-F 2 "" H 3400 4900 50  0001 C CNN
-F 3 "" H 3400 4900 50  0001 C CNN
-	1    3400 4900
+P 3700 4900
+F 0 "#PWR09" H 3700 4750 50  0001 C CNN
+F 1 "+3.3V" H 3715 5073 50  0000 C CNN
+F 2 "" H 3700 4900 50  0001 C CNN
+F 3 "" H 3700 4900 50  0001 C CNN
+	1    3700 4900
 	1    0    0    -1
 $EndComp
@@
 L power:GND #PWR06
 U 1 1 5E84D864
-P 2850 6350
-F 0 "#PWR06" H 2850 6100 50  0001 C CNN
-F 1 "GND" H 2855 6177 50  0000 C CNN
-F 2 "" H 2850 6350 50  0001 C CNN
-F 3 "" H 2850 6350 50  0001 C CNN
-	1    2850 6350
+P 2850 6550
+F 0 "#PWR06" H 2850 6300 50  0001 C CNN
+F 1 "GND" H 2855 6377 50  0000 C CNN
+F 2 "" H 2850 6550 50  0001 C CNN
+F 3 "" H 2850 6550 50  0001 C CNN
+	1    2850 6550
 	1    0    0    -1
 $EndComp
@@
 	1850 4900 2000 4900
 Wire Wire Line
-	1850 5100 1850 5950
-Wire Wire Line
-	1850 5950 2000 5950
-Connection ~ 1850 5100
-Wire Wire Line
-	1850 5950 1850 6150
-Wire Wire Line
 	1850 6150 2000 6150
-Connection ~ 1850 5950
+Wire Wire Line
+	1850 6150 1850 6350
+Wire Wire Line
+	1850 6350 2000 6350
 Wire Wire Line
 	2650 4900 2850 4900
@@
 Connection ~ 2850 5300
 Wire Wire Line
+	2650 6550 2850 6550
+Wire Wire Line
 	2650 6350 2850 6350
 Wire Wire Line
+	2850 6350 2850 6550
+Connection ~ 2850 6550
+Wire Wire Line
 	2650 6150 2850 6150
-Wire Wire Line
-	2850 6150 2850 6350
-Connection ~ 2850 6350
-Wire Wire Line
-	2650 5950 2850 5950
 $Comp
 L power:+5V #PWR01
@@
 L Device:C_Small C3
 U 1 1 5E8A194B
-P 3150 6150
-F 0 "C3" H 3242 6196 50  0000 L CNN
-F 1 "1 uF" H 3242 6105 50  0000 L CNN
-F 2 "prom:0402" H 3150 6150 50  0001 C CNN
-F 3 "~" H 3150 6150 50  0001 C CNN
-	1    3150 6150
+P 3150 6350
+F 0 "C3" H 3242 6396 50  0000 L CNN
+F 1 "1 uF" H 3242 6305 50  0000 L CNN
+F 2 "prom:0402" H 3150 6350 50  0001 C CNN
+F 3 "~" H 3150 6350 50  0001 C CNN
+	1    3150 6350
 	1    0    0    -1
 $EndComp
@@
 L power:GND #PWR08
 U 1 1 5E8A5A60
-P 3150 6350
-F 0 "#PWR08" H 3150 6100 50  0001 C CNN
-F 1 "GND" H 3155 6177 50  0000 C CNN
-F 2 "" H 3150 6350 50  0001 C CNN
-F 3 "" H 3150 6350 50  0001 C CNN
-	1    3150 6350
+P 3150 6550
+F 0 "#PWR08" H 3150 6300 50  0001 C CNN
+F 1 "GND" H 3155 6377 50  0000 C CNN
+F 2 "" H 3150 6550 50  0001 C CNN
+F 3 "" H 3150 6550 50  0001 C CNN
+	1    3150 6550
 	1    0    0    -1
 $EndComp
@@
 Connection ~ 3150 4900
 Wire Wire Line
-	3150 4900 3400 4900
+	3150 4900 3500 4900
 Wire Wire Line
 	3150 5200 3150 5300
 Wire Wire Line
-	3150 5950 3150 6050
-Connection ~ 3150 5950
-Wire Wire Line
-	3150 5950 3450 5950
-Wire Wire Line
-	3150 6250 3150 6350
+	3150 6150 3150 6250
+Connection ~ 3150 6150
+Wire Wire Line
+	3150 6150 3450 6150
+Wire Wire Line
+	3150 6450 3150 6550
 Wire Wire Line
 	1450 4900 1450 5000
@@
 $EndComp
 $Comp
-L Connector:TestPoint_Alt TP?
+L prom-rescue:TestPoint_Alt-Connector TP?
 U 1 1 5E8ADFB4
 P 2850 4900
 AR Path="/5E85CF8D/5E8ADFB4" Ref="TP?"  Part="1"
 AR Path="/5E85C2D7/5E8ADFB4" Ref="TP1"  Part="1"
+AR Path="/5E8ADFB4" Ref="TP1"  Part="1"
 F 0 "TP1" H 2750 5150 50  0000 L CNN
 F 1 "TestPoint_Alt" H 2908 4927 50  0001 L CNN
@@
 $EndComp
 $Comp
-L Connector:TestPoint_Alt TP?
+L prom-rescue:TestPoint_Alt-Connector TP?
 U 1 1 5E8B033B
-P 2850 5950
+P 2850 6150
 AR Path="/5E85CF8D/5E8B033B" Ref="TP?"  Part="1"
 AR Path="/5E85C2D7/5E8B033B" Ref="TP2"  Part="1"
-F 0 "TP2" H 2750 6200 50  0000 L CNN
-F 1 "TestPoint_Alt" H 2908 5977 50  0001 L CNN
-F 2 "prom:test-point-25" H 3050 5950 50  0001 C CNN
-F 3 "~" H 3050 5950 50  0001 C CNN
-	1    2850 5950
-	1    0    0    -1
-$EndComp
-Connection ~ 2850 5950
-Wire Wire Line
-	2850 5950 3150 5950
+AR Path="/5E8B033B" Ref="TP2"  Part="1"
+F 0 "TP2" H 2750 6400 50  0000 L CNN
+F 1 "TestPoint_Alt" H 2908 6177 50  0001 L CNN
+F 2 "prom:test-point-25" H 3050 6150 50  0001 C CNN
+F 3 "~" H 3050 6150 50  0001 C CNN
+	1    2850 6150
+	1    0    0    -1
+$EndComp
+Connection ~ 2850 6150
+Wire Wire Line
+	2850 6150 3150 6150
 Connection ~ 2850 4900
 Wire Wire Line
 	2850 4900 3150 4900
+Wire Wire Line
+	3500 4900 3500 5700
+Wire Wire Line
+	3500 5700 1550 5700
+Wire Wire Line
+	1550 5700 1550 6150
+Wire Wire Line
+	1550 6150 1850 6150
+Connection ~ 3500 4900
+Wire Wire Line
+	3500 4900 3700 4900
+Connection ~ 1850 6150
 $EndSCHEMATC

Commit message: fold the rescued schematic symbols into the local library
Parts:
- TP1, TP2: symbol prom-rescue:TestPoint_Alt-Connector -> local:TestPoint_Alt
Changed lines of the file:
@@
 $EndComp
 $Comp
-L power:GND #PWR03
+L local:GND #PWR03
 U 1 1 5E809D88
 P 1950 3250
@@
 $EndComp
 $Comp
-L power:+5V #PWR04
+L local:+5V #PWR04
 U 1 1 5E80A02F
 P 2850 2350
@@
 	5050 1550 4600 1550
 $Comp
-L power:GND #PWR012
+L local:GND #PWR012
 U 1 1 5E80C217
 P 5050 1750
@@
 $EndComp
 $Comp
-L power:+3.3V #PWR011
+L local:+3.3V #PWR011
 U 1 1 5E80C8C8
 P 5050 1250
@@
 $EndComp
 $Comp
-L power:GND #PWR014
+L local:GND #PWR014
 U 1 1 5E8116D1
 P 5050 2800
@@
 $EndComp
 $Comp
-L power:GND #PWR016
+L local:GND #PWR016
 U 1 1 5E811918
 P 5050 3850
@@
 $EndComp
 $Comp
-L power:GND #PWR018
+L local:GND #PWR018
 U 1 1 5E811B65
 P 5050 4900
@@
 $EndComp
 $Comp
-L power:+3.3V #PWR013
+L local:+3.3V #PWR013
 U 1 1 5E811DDC
 P 5050 2300
@@
 $EndComp
 $Comp
-L power:+3.3V #PWR015
+L local:+3.3V #PWR015
 U 1 1 5E81218A
 P 5050 3350
@@
 $EndComp
 $Comp
-L power:+3.3V #PWR017
+L local:+3.3V #PWR017
 U 1 1 5E8124E5
 P 5050 4400
@@
 $EndComp
 $Comp
-L power:+3.3V #PWR019
+L local:+3.3V #PWR019
 U 1 1 5E812964
 P 5050 5450
@@
 $EndComp
 $Comp
-L power:GND #PWR020
+L local:GND #PWR020
 U 1 1 5E812D10
 P 5050 5950
@@
 DIP_A2
 $Comp
-L power:+1V2 #PWR010
+L local:+1V2 #PWR010
 U 1 1 5E84CCB2
 P 3450 6150
@@
 $EndComp
 $Comp
-L power:+3.3V #PWR09
+L local:+3.3V #PWR09
 U 1 1 5E84D3A3
 P 3700 4900
@@
 $EndComp
 $Comp
-L power:GND #PWR06
+L local:GND #PWR06
 U 1 1 5E84D864
 P 2850 6550
@@
 $EndComp
 $Comp
-L power:GND #PWR05
+L local:GND #PWR05
 U 1 1 5E84DB05
 P 2850 5300
@@
 	2650 6150 2850 6150
 $Comp
-L power:+5V #PWR01
+L local:+5V #PWR01
 U 1 1 5E85C184
 P 1100 4900
@@
 $EndComp
 $Comp
-L power:GND #PWR07
+L local:GND #PWR07
 U 1 1 5E8A5808
 P 3150 5300
@@
 $EndComp
 $Comp
-L power:GND #PWR08
+L local:GND #PWR08
 U 1 1 5E8A5A60
 P 3150 6550
@@
 $EndComp
 $Comp
-L power:GND #PWR02
+L local:GND #PWR02
 U 1 1 5E8A6084
 P 1450 5250
@@
 	7700 3850 8150 3850
 $Comp
-L power:GND #PWR022
+L local:GND #PWR022
 U 1 1 5E8F110E
 P 8150 2550
@@
 $EndComp
 $Comp
-L power:GND #PWR024
+L local:GND #PWR024
 U 1 1 5E8F1499
 P 8150 4050
@@
 $EndComp
 $Comp
-L power:+3.3V #PWR021
+L local:+3.3V #PWR021
 U 1 1 5E8F17D2
 P 8150 1750
@@
 $EndComp
 $Comp
-L power:+3.3V #PWR023
+L local:+3.3V #PWR023
 U 1 1 5E8F1BEC
 P 8150 3250
@@
 $EndComp
 $Comp
-L prom-rescue:TestPoint_Alt-Connector TP?
+L local:TestPoint_Alt TP?
 U 1 1 5E8ADFB4
 P 2850 4900
@@
 $EndComp
 $Comp
-L prom-rescue:TestPoint_Alt-Connector TP?
+L local:TestPoint_Alt TP?
 U 1 1 5E8B033B
 P 2850 6150
