File: apple-1/chips/MMI-6301/kicad/prom_io_power.sch (KiCad schematic (older format))
At the start: 15 parts, among them J1 DIP16_pins, U1 TLV743P 3.3V, U2 TLV743P 1.2V, U3 74LVC2G34, U4 74LVC2G34, U5 74LVC2G34, U6 74LVC2G34, U7 74LVC2G34, U8 74LVC2G125, U9 74LVC2G125

Commit message: completed layout
Parts:
- TP1, TP2: footprint prom:test-point-25 -> prom:test-point
Changed lines of the file:
@@
 F 0 "TP1" H 2750 5150 50  0000 L CNN
 F 1 "TestPoint_Alt" H 2908 4927 50  0001 L CNN
-F 2 "prom:test-point-25" H 3050 4900 50  0001 C CNN
+F 2 "prom:test-point" H 3050 4900 50  0001 C CNN
 F 3 "~" H 3050 4900 50  0001 C CNN
 	1    2850 4900
@@
 F 0 "TP2" H 2750 6400 50  0000 L CNN
 F 1 "TestPoint_Alt" H 2908 6177 50  0001 L CNN
-F 2 "prom:test-point-25" H 3050 6150 50  0001 C CNN
+F 2 "prom:test-point" H 3050 6150 50  0001 C CNN
 F 3 "~" H 3050 6150 50  0001 C CNN
 	1    2850 6150

Commit message: library tweak
Parts:
- C1, C2, C3: symbol Device:C_Small -> local:C_Small
Changed lines of the file:
@@
 DIP_D3
 $Comp
-L Device:C_Small C1
+L local:C_Small C1
 U 1 1 5E8A0689
 P 1450 5100
@@
 $EndComp
 $Comp
-L Device:C_Small C2
+L local:C_Small C2
 U 1 1 5E8A0FD1
 P 3150 5100
@@
 $EndComp
 $Comp
-L Device:C_Small C3
+L local:C_Small C3
 U 1 1 5E8A194B
 P 3150 6350
