File: apple-1/boards/cassette-interface/kicad/cassette_interface.sch (KiCad schematic (older format))
At the start: 23 parts, among them J1 APPLE1_EDGE, J2 audio_jack, J3 audio_jack, Q1 Q_NPN_EBC, Q2 Q_NPN_EBC, U1 74LS02, U2 74LS10, U3 LM311, U4 74LS74, U5 MMI6301, U6 MMI6301

Commit message: make all symbols and footprints local; no silkscreen
Parts:
- C1: symbol Device:C_Small -> cassette:C_Small
- D1: symbol Device:LED_ALT -> cassette:LED_ALT
- Q1, Q2: symbol Device:Q_NPN_EBC -> cassette:Q_NPN_EBC
- R1, R10, R2, R3, R4, R5, R6, R7, R8, R9: symbol Device:R_US -> cassette:R_US
- U1: symbol 74xx:74LS02 -> cassette:74LS02
- U2: symbol 74xx:74LS10 -> cassette:74LS10
- U3: symbol Comparator:LM311 -> cassette:LM311-Comparator
- U4: symbol 74xx:74LS74 -> cassette:74LS74
Changed lines of the file:
@@
 $EndDescr
 $Comp
-L 74xx:74LS02 U1
+L cassette:74LS02 U1
 U 1 1 5E466DDF
 P 2800 1400
@@
 $EndComp
 $Comp
-L 74xx:74LS02 U1
+L cassette:74LS02 U1
 U 2 1 5E4686AD
 P 7700 2950
@@
 $EndComp
 $Comp
-L 74xx:74LS02 U1
+L cassette:74LS02 U1
 U 3 1 5E46965D
 P 2800 2000
@@
 $EndComp
 $Comp
-L 74xx:74LS02 U1
+L cassette:74LS02 U1
 U 4 1 5E46A99C
 P 5150 1700
@@
 $EndComp
 $Comp
-L 74xx:74LS10 U2
+L cassette:74LS10 U2
 U 1 1 5E46BCD7
 P 5900 2950
@@
 $EndComp
 $Comp
-L 74xx:74LS10 U2
+L cassette:74LS10 U2
 U 2 1 5E46CBDD
 P 4000 1700
@@
 $EndComp
 $Comp
-L 74xx:74LS10 U2
+L cassette:74LS10 U2
 U 3 1 5E46D9CF
 P 6800 2950
@@
 $EndComp
 $Comp
-L 74xx:74LS10 U2
+L cassette:74LS10 U2
 U 4 1 5E46E908
 P 9000 1450
@@
 $EndComp
 $Comp
-L 74xx:74LS74 U4
+L cassette:74LS74 U4
 U 1 1 5E47121D
 P 6300 1700
@@
 $EndComp
 $Comp
-L 74xx:74LS74 U4
+L cassette:74LS74 U4
 U 3 1 5E4721A2
 P 9800 1450
@@
 $EndComp
 $Comp
-L Comparator:LM311 U3
+L cassette:LM311-Comparator U3
 U 1 1 5E472DF2
 P 4500 3850
@@
 Apple-1 Cassette Interface
 $Comp
-L Device:Q_NPN_EBC Q1
+L cassette:Q_NPN_EBC Q1
 U 1 1 5E47FC4F
 P 4500 6150
@@
 $EndComp
 $Comp
-L Device:Q_NPN_EBC Q2
+L cassette:Q_NPN_EBC Q2
 U 1 1 5E481B80
 P 4850 6500
@@
 $EndComp
 $Comp
-L power:GND #PWR018
+L cassette:GND #PWR018
 U 1 1 5E4832C2
 P 9800 3350
@@
 $EndComp
 $Comp
-L Device:C_Small C1
+L cassette:C_Small C1
 U 1 1 5E485171
 P 3200 3850
@@
 $EndComp
 $Comp
-L power:-12V #PWR06
+L cassette:-12V #PWR06
 U 1 1 5E485E9E
 P 4400 4500
@@
 $EndComp
 $Comp
-L power:+5V #PWR02
+L cassette:+5V #PWR02
 U 1 1 5E486A44
 P 4950 5250
@@
 $EndComp
 $Comp
-L Device:LED_ALT D1
+L cassette:LED_ALT D1
 U 1 1 5E48949F
 P 4950 5700
@@
 256x4 PROM
 $Comp
-L power:GND #PWR012
+L cassette:GND #PWR012
 U 1 1 5E4B4281
 P 9000 1950
@@
 $EndComp
 $Comp
-L power:GND #PWR016
+L cassette:GND #PWR016
 U 1 1 5E4B4EBC
 P 9800 1850
@@
 $EndComp
 $Comp
-L power:GND #PWR07
+L cassette:GND #PWR07
 U 1 1 5E4B73EE
 P 7100 2200
@@
 $EndComp
 $Comp
-L power:GND #PWR08
+L cassette:GND #PWR08
 U 1 1 5E4B801F
 P 7650 2200
@@
 $EndComp
 $Comp
-L power:GND #PWR014
+L cassette:GND #PWR014
 U 1 1 5E4B8684
 P 9350 6000
@@
 $EndComp
 $Comp
-L power:GND #PWR010
+L cassette:GND #PWR010
 U 1 1 5E4B8CEC
 P 7500 6000
@@
 	2100 6700 2450 6700
 $Comp
-L 74xx:74LS02 U1
+L cassette:74LS02 U1
 U 5 1 5E4701AC
 P 9800 2850
@@
 $EndComp
 $Comp
-L Device:R_US R2
+L cassette:R_US R2
 U 1 1 5E575731
 P 4950 5400
@@
 	4600 6500 4650 6500
 $Comp
-L power:GND #PWR03
+L cassette:GND #PWR03
 U 1 1 5E4B6154
 P 4950 6700
@@
 $EndComp
 $Comp
-L Device:R_US R10
+L cassette:R_US R10
 U 1 1 5E626D5F
 P 7100 2050
@@
 $EndComp
 $Comp
-L Device:R_US R9
+L cassette:R_US R9
 U 1 1 5E627816
 P 7100 1750
@@
 	6600 1600 7100 1600
 $Comp
-L Device:R_US R1
+L cassette:R_US R1
 U 1 1 5E66C320
 P 4150 6150
@@
 $EndComp
 $Comp
-L Device:R_US R3
+L cassette:R_US R3
 U 1 1 5E676CC2
 P 3450 3450
@@
 $EndComp
 $Comp
-L Device:R_US R4
+L cassette:R_US R4
 U 1 1 5E677AC2
 P 3450 4300
@@
 $EndComp
 $Comp
-L Device:R_US R5
+L cassette:R_US R5
 U 1 1 5E6782D1
 P 3800 3450
@@
 $EndComp
 $Comp
-L Device:R_US R6
+L cassette:R_US R6
 U 1 1 5E678C01
 P 3800 4300
@@
 $EndComp
 $Comp
-L Device:R_US R8
+L cassette:R_US R8
 U 1 1 5E67941E
 P 5000 4000
@@
 $EndComp
 $Comp
-L Device:R_US R7
+L cassette:R_US R7
 U 1 1 5E679B6C
 P 5000 3600
@@
 $EndComp
 $Comp
-L power:GND #PWR04
+L cassette:GND #PWR04
 U 1 1 5E68922B
 P 4000 4450
@@
 $EndComp
 $Comp
-L power:+5V #PWR05
+L cassette:+5V #PWR05
 U 1 1 5E689A79
 P 4150 3300
@@
 -12V
 $Comp
-L power:+5V #PWR09
+L cassette:+5V #PWR09
 U 1 1 5E6F9E6D
 P 7500 4600
@@
 $EndComp
 $Comp
-L power:+5V #PWR013
+L cassette:+5V #PWR013
 U 1 1 5E6FA7E1
 P 9350 4600
@@
 PROM_A0
 $Comp
-L power:+5V #PWR017
+L cassette:+5V #PWR017
 U 1 1 5E7E0781
 P 9800 2350
@@
 $EndComp
 $Comp
-L power:+5V #PWR015
+L cassette:+5V #PWR015
 U 1 1 5E7E0D97
 P 9800 1050
@@
 $EndComp
 $Comp
-L power:+5V #PWR011
+L cassette:+5V #PWR011
 U 1 1 5E7E12A4
 P 9000 950
@@
 NoConn ~ 4600 3550
 $Comp
-L power:GND #PWR01
+L cassette:GND #PWR01
 U 1 1 5E84F1F0
 P 2800 4150
